Commit message: fixed octomap problem

File: semantic_maps/urdf/lucrezio.urdf.xacro (robot description, xacro)
@@ -17,9 +17,9 @@
       </geometry>
     </visual>
-    <collision>
+    <!--<collision>
       <geometry>
         <box size="${base_length} ${base_width} ${base_height}"/>
       </geometry>
-    </collision>
+    </collision>-->
     <visual>
       <origin xyz="-${base_length/2 - base_height/2} 0 -${base_height/2}" rpy="0 0 0" />
@@ -132,5 +132,5 @@
   <!-- LASER -->
   <link name="laser_link">
-    <collision>
+    <!--<collision>
       <origin xyz="0 0 0" rpy="0 0 0" />
       <geometry>
@@ -143,5 +143,5 @@
         <mesh filename="package://semantic_maps/meshes/hokuyo.dae" />
       </geometry>
-    </visual>
+    </visual>-->
     <inertial>
       <mass value="1e-5" />
@@ -153,5 +153,5 @@
   <joint name="laser_joint" type="fixed">
     <axis xyz="0 1 0" />
-    <origin xyz="0.1 0 0.1" rpy="0 0 0" />
+    <origin xyz="0.1 0 -0.05" rpy="0 0 0" />
     <parent link="base_link" />
     <child  link="laser_link" />
@@ -159,10 +159,10 @@
   <!-- HOKUYO SENSOR -->
   <gazebo reference="laser_link">
-    <sensor type="gpu_ray" name="head_hokuyo_sensor">
+    <sensor type="ray" name="head_hokuyo_sensor">
       <pose>0 0 0 0 0 0</pose>
       <visualize>false</visualize>
       <update_rate>40</update_rate>
       <ray>
-        <scan>
+        <!--<scan>
           <horizontal>
             <samples>1024</samples>
@@ -171,8 +171,16 @@
             <max_angle>1.57</max_angle>
           </horizontal>
+        </scan>-->
+        <scan>
+          <horizontal>
+            <samples>512</samples>
+            <resolution>1</resolution>
+            <min_angle>-1.571</min_angle>
+            <max_angle>1.571</max_angle>
+          </horizontal>
         </scan>
         <range>
-          <min>0.02</min>
-          <max>10.0</max>
+          <min>0.20</min>
+          <max>15.0</max>
           <resolution>0.01</resolution>
         </range>
@@ -183,22 +191,25 @@
         </noise>
       </ray>
-      <plugin name="gazebo_ros_head_hokuyo_controller" filename="libgazebo_ros_gpu_laser.so">
+      <plugin name="gazebo_ros_head_hokuyo_controller" filename="libgazebo_ros_laser.so">
         <topicName>/scan</topicName>
         <frameName>laser_link</frameName>
       </plugin>
     </sensor>
-  </gazebo>
+  </gazebo> -->
   <!-- CAMERA -->
   <link name="camera_link">
-    <collision>
-      <origin xyz="0 0 0" rpy="0 0 0"/>
-      <geometry>
-    <box size="${camera_link} ${camera_link} ${camera_link}"/>
-      </geometry>
-    </collision>
-    <visual>
-      <origin xyz="0 0 0" rpy="0 0 0"/>
-      <geometry>
-    <box size="${camera_link} ${camera_link} ${camera_link}"/>
+    <!--<collision>
+      <origin xyz="0 0 0" rpy="0 0 0"/>
+      <geometry>
+        <box size="${camera_link} ${camera_link} ${camera_link}"/>
+      </geometry>
+    </collision>-->
+    <visual>
+      <origin xyz="0 0 0" rpy="0 0 0"/>
+      <geometry>
+        <box size="${camera_link} ${camera_link} ${camera_link}"/>
+<!--
+<mesh filename="package://semantic_maps/meshes/kinect.dae" />
+-->
       </geometry>
       <material name="red"/>
@@ -211,9 +222,9 @@
   </link>
   <!-- CAMERA JOINT -->
-  <joint name="camera_joint" type="continuous">
-    <axis xyz="0 1 0" />
-    <origin xyz="0 0 1.0" rpy="0 0 0"/>
+  <joint name="camera_joint" type="fixed">
     <parent link="base_link"/>
     <child link="camera_link"/>
+    <axis xyz="0 1 0" />
+    <origin xyz="0 0 0.5" rpy="0 0 0"/>
   </joint>
 <!--
@@ -221,4 +232,5 @@
     <preserveFixedJoint>true</preserveFixedJoint>
   </gazebo>"
+<origin xyz="0.21 0 0.1" rpy="0 0 0"/>
 -->
   <!-- XTION SENSOR -->
@@ -226,10 +238,10 @@
     <sensor type="depth" name="rgbd_camera">
       <always_on>true</always_on>
-      <update_rate>20.0</update_rate>
+      <update_rate>30.0</update_rate>
       <camera>
         <horizontal_fov>${60.0*M_PI/180.0}</horizontal_fov>
         <image>
-          <width>320</width>
-          <height>240</height>
+          <width>640</width>
+          <height>480</height>
           <format>R8G8B8</format>
         </image>
@@ -240,7 +252,7 @@
       </camera>
       <plugin name="rgdb_camera_controller" filename="libgazebo_ros_openni_kinect.so">
-        <cameraName>camera</cameraName>
+	  <cameraName>camera</cameraName>
           <alwaysOn>true</alwaysOn>
-          <updateRate>10</updateRate>
+          <updateRate>30</updateRate>
           <imageTopicName>rgb/image_raw</imageTopicName>
           <depthImageTopicName>depth/image_raw</depthImageTopicName>
@@ -255,5 +267,5 @@
           <distortion_t1>0.0</distortion_t1>
           <distortion_t2>0.0</distortion_t2>
-          <pointCloudCutoff>0.4</pointCloudCutoff>
+	  <pointCloudCutoff>0.4</pointCloudCutoff>
       </plugin>
     </sensor>

File: semantic_maps/urdf/lucrezio_with_logical.urdf.xacro (robot description, xacro)
@@ -315,5 +315,5 @@
   <gazebo reference="logical_camera_link">
       <sensor name="logical_camera" type="logical_camera">
-        <plugin name="logical_camera_plugin" filename="liblogical_camera_plugin.so"/>
+         <plugin name="logical_camera_plugin" filename="liblogical_camera_plugin.so"/>
           <logical_camera>
             <near>0.02</near>

File: semantic_maps/urdf/lucrezio_with_logical_noLaser.urdf.xacro (robot description, xacro)
@@ -310,5 +310,5 @@
             <far>8.0</far>
             <horizontal_fov>${60.0*M_PI/180.0}</horizontal_fov>
-            <aspect_ratio>1.778</aspect_ratio>
+           <!-- <aspect_ratio>1.778</aspect_ratio> -->
           </logical_camera>
           <visualize>false</visualize>
@@ -316,4 +316,6 @@
           <update_rate>20</update_rate>
       </sensor>
+  </gazebo>
+  <gazebo>
   </gazebo>
   <!-- Gazebo plugin for ROS Control -->
