Commit message: integrated yolo5 with object_detection_node

File: semantic_maps/urdf/new_robot.urdf.xacro (robot description, xacro)
@@ -2,4 +2,5 @@
 <robot xmlns:xacro="http://www.ros.org/wiki/xacro" name="robot">
   <!-- CONSTANTS -->
+  <xacro:property name="height" value="0.5" />
   <xacro:property name="base_length" value="0.4" />
   <xacro:property name="base_width" value="0.2" />
@@ -13,15 +14,16 @@
   <link name="base_link">
     <visual>
+      <origin xyz="0 0 0.2" rpy="0 0 0" />
+      <geometry>
+        <box size="${base_length} ${base_width} ${height}"/>
+      </geometry>
+    </visual>
+    <!--<collision>
       <geometry>
         <box size="${base_length} ${base_width} ${base_height}"/>
       </geometry>
-    </visual>
-    <!--<collision>
-      <geometry>
-        <box size="${base_length} ${base_width} ${base_height}"/>
-      </geometry>
     </collision>-->
     <visual>
-      <origin xyz="-${base_length/2 - base_height/2} 0 -${base_height/2}" rpy="0 0 0" />
+      <origin xyz="0 0 -${base_height/2}" rpy="0 0 0" />
       <geometry>
         <sphere radius="${base_height/2}" />
@@ -29,5 +31,5 @@
     </visual>
     <collision>
-      <origin xyz="-${base_length/2 - base_height/2} 0 -${base_height/2}" rpy="0 0 0" />
+      <origin xyz="0 0 -${base_height/2}" rpy="0 0 0" />
       <geometry>
         <sphere radius="${base_height/2}" />
@@ -213,5 +215,4 @@
         <mesh filename="package://semantic_maps/meshes/kinect.dae" />
       </geometry>
-      <material name="red"/>
     </visual>
     <inertial>
@@ -226,5 +227,5 @@
     <child link="camera_link"/>
     <axis xyz="0 1 0" />
-    <origin xyz="0.21 0 0.5" rpy="0 0 0"/>
+    <origin xyz="0.21 0 0.503" rpy="0 0 0"/>
   </joint>
 <!--

Commit message: added evaluation_node

File: semantic_maps/urdf/new_robot.urdf.xacro (robot description, xacro)
@@ -8,5 +8,5 @@
   <xacro:property name="wheel_length" value="0.05" />
   <xacro:property name="wheel_radius" value="0.1" />
-  <xacro:property name="camera_link" value="0.05" />
+  <xacro:property name="camera_size" value="0.05" />
   <xacro:property name="camera_name" value="xtion" />
   <xacro:property name="M_PI" value="3.1415926535897931" />
@@ -134,8 +134,8 @@
   <!-- LASER -->
   <link name="laser_link">
-    <!--<collision>
+    <collision>
       <origin xyz="0 0 0" rpy="0 0 0" />
       <geometry>
-        <box size="0.1 0.1 0.1" />
+        <mesh filename="package://semantic_maps/meshes/hokuyo.dae" />
       </geometry>
     </collision>
@@ -145,5 +145,5 @@
         <mesh filename="package://semantic_maps/meshes/hokuyo.dae" />
       </geometry>
-    </visual>-->
+    </visual>
     <inertial>
       <mass value="1e-5" />
@@ -155,5 +155,5 @@
   <joint name="laser_joint" type="fixed">
     <axis xyz="0 1 0" />
-    <origin xyz="0.1 0 -0.05" rpy="0 0 0" />
+    <origin xyz="0.18 0 0.555" rpy="0 0 0" />
     <parent link="base_link" />
     <child  link="laser_link" />
@@ -272,4 +272,47 @@
     </sensor>
   </gazebo>
+  <!-- LOGICAL CAMERA -->
+  <link name="logical_camera_link">
+    <!--<collision>
+      <origin xyz="0 0 0" rpy="0 0 0"/>
+      <geometry>
+    	<mesh filename="package://semantic_maps/meshes/kinect.dae" />
+      </geometry>
+    </collision>
+    <visual>
+      <origin xyz="0 0 0" rpy="0 0 0"/>
+      <geometry>
+    	<mesh filename="package://semantic_maps/meshes/kinect.dae" />
+      </geometry>
+      <material name="red"/>
+    </visual>
+    <inertial>
+      <mass value="1e-5" />
+      <origin xyz="0 0 0" rpy="0 0 0"/>
+      <inertia ixx="1e-6" ixy="0" ixz="0" iyy="1e-6" iyz="0" izz="1e-6" />
+    </inertial>-->
+  </link>
+  <!-- LOGICAL CAMERA JOINT -->
+  <joint name="logical_camera_joint" type="fixed">
+    <axis xyz="0 1 0" />
+    <origin xyz="0.21 0 0.503" rpy="0 0 0"/>
+    <parent link="base_link"/>
+    <child link="logical_camera_link"/>
+  </joint>
+  <!-- LOGICAL CAMERA SENSOR -->
+  <gazebo reference="logical_camera_link">
+      <sensor name="logical_camera" type="logical_camera">
+         <plugin name="logical_camera_plugin" filename="liblogical_camera_plugin.so"/>
+          <logical_camera>
+            <near>0.02</near>
+            <far>8.0</far>
+            <horizontal_fov>${60.0*M_PI/180.0}</horizontal_fov>
+            <aspect_ratio>1.778</aspect_ratio>
+          </logical_camera>
+          <visualize>false</visualize>
+          <always_on>true</always_on>
+          <update_rate>20</update_rate>
+      </sensor>
+  </gazebo>
   <!-- Gazebo plugin for ROS Control -->
   <gazebo>

Commit message: fixed logical camera detection

File: semantic_maps/urdf/new_robot.urdf.xacro (robot description, xacro)
@@ -145,5 +145,5 @@
         <mesh filename="package://semantic_maps/meshes/hokuyo.dae" />
       </geometry>
-    </visual>
+    </visual>-->
     <inertial>
       <mass value="1e-5" />
@@ -204,5 +204,5 @@
       <origin xyz="0 0 0" rpy="0 0 0"/>
       <geometry>
-        <box size="${camera_link} ${camera_link} ${camera_link}"/>
+        <mesh filename="package://semantic_maps/meshes/kinect.dae" />
       </geometry>
     </collision>-->
@@ -274,5 +274,5 @@
   <!-- LOGICAL CAMERA -->
   <link name="logical_camera_link">
-    <!--<collision>
+    <!--collision>
       <origin xyz="0 0 0" rpy="0 0 0"/>
       <geometry>
@@ -305,8 +305,10 @@
          <plugin name="logical_camera_plugin" filename="liblogical_camera_plugin.so"/>
           <logical_camera>
-            <near>0.02</near>
-            <far>8.0</far>
-            <horizontal_fov>${60.0*M_PI/180.0}</horizontal_fov>
-            <aspect_ratio>1.778</aspect_ratio>
+            <near>2.0</near>
+            <far>2.0</far>
+            <horizontal_fov>0.4</horizontal_fov>
+            <aspect_ratio>1.1</aspect_ratio>
+            <!--<horizontal_fov>${60.0*M_PI/180.0}</horizontal_fov>
+            <aspect_ratio>1.778</aspect_ratio>-->
           </logical_camera>
           <visualize>false</visualize>

Commit message: updated new_robot.urdf

File: semantic_maps/urdf/new_robot.urdf.xacro (robot description, xacro)
@@ -2,10 +2,11 @@
 <robot xmlns:xacro="http://www.ros.org/wiki/xacro" name="robot">
   <!-- CONSTANTS -->
-  <xacro:property name="height" value="0.5" />
+  <xacro:property name="height" value="0.4" />
   <xacro:property name="base_length" value="0.4" />
-  <xacro:property name="base_width" value="0.2" />
+  <xacro:property name="base_width" value="0.35" />
   <xacro:property name="base_height" value="0.1" />
   <xacro:property name="wheel_length" value="0.05" />
   <xacro:property name="wheel_radius" value="0.1" />
+  <xacro:property name="caster_radius" value="0.06" />
   <xacro:property name="camera_size" value="0.05" />
   <xacro:property name="camera_name" value="xtion" />
@@ -14,5 +15,5 @@
   <link name="base_link">
     <visual>
-      <origin xyz="0 0 0.2" rpy="0 0 0" />
+      <origin xyz="0 0 0.25" rpy="0 0 0" />
       <geometry>
         <box size="${base_length} ${base_width} ${height}"/>
@@ -25,17 +26,17 @@
     </collision>-->
     <visual>
-      <origin xyz="0 0 -${base_height/2}" rpy="0 0 0" />
-      <geometry>
-        <sphere radius="${base_height/2}" />
+      <origin xyz="-0.14 0 -${base_height/2-0.02}" rpy="0 0 0" />
+      <geometry>
+        <sphere radius="0.075" />
       </geometry>
     </visual>
     <collision>
-      <origin xyz="0 0 -${base_height/2}" rpy="0 0 0" />
-      <geometry>
-        <sphere radius="${base_height/2}" />
-      </geometry>
-    </collision>
-    <inertial>
-      <mass value="0.6"/>
+      <origin xyz="-0.14 0 -${base_height/2-0.02}" rpy="0 0 0" />
+      <geometry>
+        <sphere radius="0.075" />
+      </geometry>
+    </collision>
+    <inertial>
+      <mass value="3.6"/>
       <inertia ixx="1e-3" ixy="0.0" ixz="0.0" iyy="1e-3" iyz="0.0" izz="1e-3"/>
     </inertial>
@@ -61,5 +62,5 @@
     </collision>
     <inertial>
-      <mass value="0.6"/>
+      <mass value="3.6"/>
       <inertia ixx="1e-3" ixy="0.0" ixz="0.0" iyy="1e-3" iyz="0.0" izz="1e-3"/>
     </inertial>
@@ -76,5 +77,5 @@
     <parent link="base_link" />
     <child  link="left_wheel" />
-    <origin xyz="0.1 0.13 0" />
+    <origin xyz="0.1 0.20 0" />
     <axis rpy="0 0 0" xyz="0 1 0"/>
   </joint>
@@ -104,5 +105,5 @@
     </collision>
     <inertial>
-      <mass value="0.6"/>
+      <mass value="3.6"/>
       <inertia ixx="1e-3" ixy="0.0" ixz="0.0" iyy="1e-3" iyz="0.0" izz="1e-3"/>
     </inertial>
@@ -119,5 +120,5 @@
     <parent link="base_link" />
     <child  link="right_wheel" />
-    <origin xyz="0.1 -0.13 0" />
+    <origin xyz="0.1 -0.20 0" />
     <axis rpy="0 0 0" xyz="0 1 0"/>
   </joint>
